File: GaN_Leistungsplatine_V3.kicad_pcb (KiCad board)
At the start: 4 copper layers, 100 x 100 mm, 91 parts, among them J1 GPI0_1, J10 Conn_02x02_Top_Bottom, J2 105-1102-001, J3 105-1102-001, J4 105-1102-001, J5 105-1102-001, J6 105-1102-001, J7 105-1102-001, J8 105-1102-001, J9 Conn_02x03_Counter_Clockwise, Q1 GaN_FET_with_Source_Kelvin_Pin, Q2 GaN_FET_with_Source_Kelvin_Pin, U1 LT1999, U2 NCP51810

Commit message: hello
Parts:
- moved C29 7.08 mm to (79.9, 106.2), turned to 135 degrees
- moved R6 5.70 mm to (74.9, 102.5), turned to -135 degrees
- moved C28 4.15 mm to (78.6, 107.5), turned to 135 degrees
- moved R8 4.10 mm to (76.1, 105.0), turned to -45 degrees
- moved D1 3.72 mm to (71.6, 100.5), turned to -135 degrees
- moved R7 2.61 mm to (75.4, 113.0), turned to 45 degrees
- moved C23 2.09 mm to (81.1, 105.0), turned to -45 degrees
- moved C27 1.68 mm to (74.1, 111.7), turned to 45 degrees

Commit message: platinen change
Parts:
- moved C7 11.4 mm to (32.8, 80.6)
Changed lines of the file:
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@@
     (48 "B.Fab" user)
     (49 "F.Fab" user)
-    (50 "User.1" user)
-    (51 "User.2" user)
-    (52 "User.3" user)
-    (53 "User.4" user)
-    (54 "User.5" user)
-    (55 "User.6" user)
-    (56 "User.7" user)
-    (57 "User.8" user)
-    (58 "User.9" user)
+    (50 "User.1" user "Nutzer.1")
+    (51 "User.2" user "Nutzer.2")
+    (52 "User.3" user "Nutzer.3")
+    (53 "User.4" user "Nutzer.4")
+    (54 "User.5" user "Nutzer.5")
+    (55 "User.6" user "Nutzer.6")
+    (56 "User.7" user "Nutzer.7")
+    (57 "User.8" user "Nutzer.8")
+    (58 "User.9" user "Nutzer.9")
   )
   (setup
@@
   )
   (footprint "Capacitor_SMD:C_1206_3216Metric_Pad1.33x1.80mm_HandSolder" (layer "F.Cu")
-    (at 35.13 91.73)
+    (at 32.75 80.61)
     (descr "Capacitor SMD 1206 (3216 Metric), square (rectangular) end terminal, IPC_7351 nominal with elongated pad for handsoldering. (Body size source: IPC-SM-782 page 76, https://www.pcb-3d.com/wordpress/wp-content/uploads/ipc-sm-782a_amendment_1_and_2.pdf), generated with kicad-footprint-generator")
     (tags "capacitor handsolder")
